File: Kicad-Files/TinyFox V2.sch (KiCad schematic (older format))
At the start: 6 parts

Commit message: Add files via upload
Parts:
- added C?: 100nF, symbol Device:C
- C?: value 100nF -> 100pF
Connections:
- net labels removed: +3.3V
- wire segments 41 -> 48
Changed lines of the file:
@@
 	-1   0    0    1
-$EndComp
-$Comp
-L power:+3.3V #PWR?
-U 1 1 6140291F
-P 4050 3500
-F 0 "#PWR?" H 4050 3350 50  0001 C CNN
-F 1 "+3.3V" H 4065 3673 50  0000 C CNN
-F 2 "" H 4050 3500 50  0001 C CNN
-F 3 "" H 4050 3500 50  0001 C CNN
-	1    4050 3500
-	1    0    0    -1
 $EndComp
 Wire Wire Line
@@
 RST
 Wire Wire Line
-	5450 2650 5450 2750
+	5450 2500 5450 2600
 $Comp
 L power:GND #PWR?
@@
 P 6950 3350
 F 0 "C?" V 6698 3350 50  0000 C CNN
-F 1 "100nF" V 6789 3350 50  0000 C CNN
+F 1 "100pF" V 6789 3350 50  0000 C CNN
 F 2 "" H 6988 3200 50  0001 C CNN
 F 3 "~" H 6950 3350 50  0001 C CNN
@@
 L power:VCC #PWR?
 U 1 1 613DBF72
-P 5450 2650
-F 0 "#PWR?" H 5450 2500 50  0001 C CNN
-F 1 "VCC" H 5465 2823 50  0000 C CNN
-F 2 "" H 5450 2650 50  0001 C CNN
-F 3 "" H 5450 2650 50  0001 C CNN
-	1    5450 2650
+P 5450 2500
+F 0 "#PWR?" H 5450 2350 50  0001 C CNN
+F 1 "VCC" H 5465 2673 50  0000 C CNN
+F 2 "" H 5450 2500 50  0001 C CNN
+F 3 "" H 5450 2500 50  0001 C CNN
+	1    5450 2500
 	1    0    0    -1
 $EndComp
@@
 EndData
 $EndBitmap
+$Comp
+L Device:C C?
+U 1 1 613BE0DC
+P 5800 2600
+F 0 "C?" V 5548 2600 50  0000 C CNN
+F 1 "100nF" V 5639 2600 50  0000 C CNN
+F 2 "" H 5838 2450 50  0001 C CNN
+F 3 "~" H 5800 2600 50  0001 C CNN
+	1    5800 2600
+	0    -1   -1   0
+$EndComp
+Wire Wire Line
+	5650 2600 5450 2600
+Connection ~ 5450 2600
+Wire Wire Line
+	5450 2600 5450 2750
+$Comp
+L power:GND #PWR?
+U 1 1 613C0D8B
+P 7800 2950
+F 0 "#PWR?" H 7800 2700 50  0001 C CNN
+F 1 "GND" H 7805 2777 50  0000 C CNN
+F 2 "" H 7800 2950 50  0001 C CNN
+F 3 "" H 7800 2950 50  0001 C CNN
+	1    7800 2950
+	1    0    0    -1
+$EndComp
+Wire Wire Line
+	7700 2650 7800 2650
+Wire Wire Line
+	7800 2650 7800 2850
+Wire Wire Line
+	7700 2850 7800 2850
+Connection ~ 7800 2850
+Wire Wire Line
+	7800 2850 7800 2950
+$Comp
+L power:GND #PWR?
+U 1 1 613C294C
+P 6150 2600
+F 0 "#PWR?" H 6150 2350 50  0001 C CNN
+F 1 "GND" H 6155 2427 50  0000 C CNN
+F 2 "" H 6150 2600 50  0001 C CNN
+F 3 "" H 6150 2600 50  0001 C CNN
+	1    6150 2600
+	0    -1   -1   0
+$EndComp
+Wire Wire Line
+	5950 2600 6150 2600
+$Comp
+L power:VCC #PWR?
+U 1 1 613C4449
+P 4050 3500
+F 0 "#PWR?" H 4050 3350 50  0001 C CNN
+F 1 "VCC" H 4065 3673 50  0000 C CNN
+F 2 "" H 4050 3500 50  0001 C CNN
+F 3 "" H 4050 3500 50  0001 C CNN
+	1    4050 3500
+	1    0    0    -1
+$EndComp
 $EndSCHEMATC

Commit message: Add files via upload
Parts:
- gave numbers to parts that had none: 7
Changed lines of the file:
@@
 $EndDescr
 $Comp
-L Modulos:SIGFOX_WISOL_RC4 U?
+L Modulos:SIGFOX_WISOL_RC4 U1
 U 1 1 61614F6C
 P 3550 5150
-F 0 "U?" H 6300 7400 50  0000 C CNN
+F 0 "U1" H 6300 7400 50  0000 C CNN
 F 1 "SIGFOX_WISOL_RC4" H 4900 7400 50  0000 C CNN
 F 2 "" H 3550 5150 50  0001 C CNN
@@
 NoConn ~ 4350 4450
 $Comp
-L Device:R_US R?
+L Device:R_US R1
 U 1 1 6140147A
 P 4050 3800
-F 0 "R?" H 3982 3754 50  0000 R CNN
+F 0 "R1" H 3982 3754 50  0000 R CNN
 F 1 "10K" H 3982 3845 50  0000 R CNN
 F 2 "" V 4090 3790 50  0001 C CNN
@@
 	5450 2500 5450 2600
 $Comp
-L power:GND #PWR?
+L power:GND #PWR02
 U 1 1 6141CDF9
 P 5350 5150
-F 0 "#PWR?" H 5350 4900 50  0001 C CNN
+F 0 "#PWR02" H 5350 4900 50  0001 C CNN
 F 1 "GND" H 5355 4977 50  0000 C CNN
 F 2 "" H 5350 5150 50  0001 C CNN
@@
 	5750 5050 5650 5050
 $Comp
-L Device:C C?
+L Device:C C2
 U 1 1 6146F34A
 P 6950 3350
-F 0 "C?" V 6698 3350 50  0000 C CNN
+F 0 "C2" V 6698 3350 50  0000 C CNN
 F 1 "100pF" V 6789 3350 50  0000 C CNN
 F 2 "" H 6988 3200 50  0001 C CNN
@@
 $EndComp
 $Comp
-L Device:Antenna AE?
+L Device:Antenna AE1
 U 1 1 6147069C
 P 7700 3350
-F 0 "AE?" V 7654 3480 50  0000 L CNN
+F 0 "AE1" V 7654 3480 50  0000 L CNN
 F 1 "Antenna" V 7745 3480 50  0000 L CNN
 F 2 "" H 7700 3350 50  0001 C CNN
@@
 NoConn ~ 6550 4250
 $Comp
-L Mis~Conectores:1909763-1 J?
+L Mis~Conectores:1909763-1 J2
 U 1 1 614E88DF
 P 7300 3150
-F 0 "J?" H 7408 3915 50  0000 C CNN
+F 0 "J2" H 7408 3915 50  0000 C CNN
 F 1 "1909763-1" H 7408 3824 50  0000 C CNN
 F 2 "TE_Connectivity-1909763-1-*" H 7300 4000 50  0001 L CNN
@@
 	7300 3350 7500 3350
 $Comp
-L Connector:Conn_01x06_Male J?
+L Connector:Conn_01x06_Male J1
 U 1 1 613D13DE
 P 7100 5250
-F 0 "J?" V 7254 4862 50  0000 R CNN
+F 0 "J1" V 7254 4862 50  0000 R CNN
 F 1 "Conn_01x06_Male" V 7163 4862 50  0000 R CNN
 F 2 "" H 7100 5250 50  0001 C CNN
@@
 	6550 3350 6800 3350
 $Comp
-L power:GND #PWR?
+L power:GND #PWR05
 U 1 1 613D8ECD
 P 6700 4800
-F 0 "#PWR?" H 6700 4550 50  0001 C CNN
+F 0 "#PWR05" H 6700 4550 50  0001 C CNN
 F 1 "GND" H 6705 4627 50  0000 C CNN
 F 2 "" H 6700 4800 50  0001 C CNN
@@
 $EndComp
 $Comp
-L power:GND #PWR?
+L power:GND #PWR07
 U 1 1 613DA8D3
 P 7600 4800
-F 0 "#PWR?" H 7600 4550 50  0001 C CNN
+F 0 "#PWR07" H 7600 4550 50  0001 C CNN
 F 1 "GND" H 7605 4627 50  0000 C CNN
 F 2 "" H 7600 4800 50  0001 C CNN
@@
 $EndComp
 $Comp
-L power:VCC #PWR?
+L power:VCC #PWR06
 U 1 1 613DB0E7
 P 7000 4850
-F 0 "#PWR?" H 7000 4700 50  0001 C CNN
+F 0 "#PWR06" H 7000 4700 50  0001 C CNN
 F 1 "VCC" H 7015 5023 50  0000 C CNN
 F 2 "" H 7000 4850 50  0001 C CNN
@@
 $EndComp
 $Comp
-L power:VCC #PWR?
+L power:VCC #PWR03
 U 1 1 613DBF72
 P 5450 2500
-F 0 "#PWR?" H 5450 2350 50  0001 C CNN
+F 0 "#PWR03" H 5450 2350 50  0001 C CNN
 F 1 "VCC" H 5465 2673 50  0000 C CNN
 F 2 "" H 5450 2500 50  0001 C CNN
@@
 $EndBitmap
 $Comp
-L Device:C C?
+L Device:C C1
 U 1 1 613BE0DC
 P 5800 2600
-F 0 "C?" V 5548 2600 50  0000 C CNN
+F 0 "C1" V 5548 2600 50  0000 C CNN
 F 1 "100nF" V 5639 2600 50  0000 C CNN
 F 2 "" H 5838 2450 50  0001 C CNN
@@
 	5450 2600 5450 2750
 $Comp
-L power:GND #PWR?
+L power:GND #PWR08
 U 1 1 613C0D8B
 P 7800 2950
-F 0 "#PWR?" H 7800 2700 50  0001 C CNN
+F 0 "#PWR08" H 7800 2700 50  0001 C CNN
 F 1 "GND" H 7805 2777 50  0000 C CNN
 F 2 "" H 7800 2950 50  0001 C CNN
@@
 	7800 2850 7800 2950
 $Comp
-L power:GND #PWR?
+L power:GND #PWR04
 U 1 1 613C294C
 P 6150 2600
-F 0 "#PWR?" H 6150 2350 50  0001 C CNN
+F 0 "#PWR04" H 6150 2350 50  0001 C CNN
 F 1 "GND" H 6155 2427 50  0000 C CNN
 F 2 "" H 6150 2600 50  0001 C CNN
@@
 	5950 2600 6150 2600
 $Comp
-L power:VCC #PWR?
+L power:VCC #PWR01
 U 1 1 613C4449
 P 4050 3500
-F 0 "#PWR?" H 4050 3350 50  0001 C CNN
+F 0 "#PWR01" H 4050 3350 50  0001 C CNN
 F 1 "VCC" H 4065 3673 50  0000 C CNN
 F 2 "" H 4050 3500 50  0001 C CNN
